Commit message: personal change to fix my expr

File: nexus_4wd_mecanum_description/urdf/nexus_4wd_mecanum.xacro (robot description, xacro)
@@ -1,11 +1,26 @@
 <?xml version="1.0"?>
-<robot name="nexus_4wd_mecanum" xmlns:xacro="http://ros.org/wiki/xacro">
+<robot name="nexus_4wd_mecanum"
+  xmlns:xacro="http://ros.org/wiki/xacro">
+  <xacro:property name="namespace" value="$(arg namespace)"/>
   <xacro:property name="PI" value="3.1415926535897931" />
   <xacro:property name="wheel_radius" value="0.050" />
   <xacro:property name="wheel_width" value="0.0505" />
-  <material name="yellow"><color rgba="0.8 0.8 0.0 1.0" /></material>
-  <material name="black"><color rgba="0.15 0.15 0.15 1.0" /></material>
-  <material name="dark_grey"><color rgba="0.2 0.2 0.2 1.0" /></material>
-  <material name="light_grey"><color rgba="0.4 0.4 0.4 1.0" /></material>
+  <xacro:property name="rplidar_offset_x" value="0.07" />
+  <xacro:property name="rplidar_offset_y" value="0.0" />
+  <xacro:property name="rplidar_offset_z" value="0.072" />
+  <material name="yellow">
+    <color rgba="0.8 0.8 0.0 1.0" />
+  </material>
+  <material name="black">
+    <color rgba="0.15 0.15 0.15 1.0" />
+  </material>
+  <material name="dark_grey">
+    <color rgba="0.2 0.2 0.2 1.0" />
+  </material>
+  <material name="light_grey">
+    <color rgba="0.4 0.4 0.4 1.0" />
+  </material>
+  <xacro:include filename="$(find nexus_4wd_mecanum_description)/urdf/imu.xacro"/>
+  <xacro:include filename="$(find nexus_4wd_mecanum_description)/urdf/livox_mid360.xacro"/>
   <link name="base_footprint"></link>
   <joint name="base_link_joint" type="fixed">
@@ -32,10 +47,19 @@
       <origin xyz="-0.01103 0 0.002" rpy="0 0 0"/>
       <mass value="2.844"/>
-      <inertia
-        ixx="0.018819942" ixy="0" ixz="-0.000101519"
-        iyy="0.057333716" iyz="0"
-        izz="0.074201740"/>
-    </inertial>
-  </link>
+      <inertia ixx="0.018819942" ixy="0" ixz="-0.000101519" iyy="0.057333716" iyz="0" izz="0.074201740"/>
+    </inertial>
+  </link>
+  <xacro:laser_livox NS="${namespace}"/>
+  <joint name="laser_joint" type="fixed">
+    <origin xyz="${rplidar_offset_x} ${rplidar_offset_y} ${rplidar_offset_z}" rpy="0 0 0" />
+    <parent link="base_link"/>
+    <child link="laser_link"/>
+  </joint>
+  <xacro:imu prefix="imu"/>
+  <joint name="imu_joint" type="fixed">
+    <origin xyz="0 0 0.0275" rpy="0 0 0" />
+    <parent link="base_link"/>
+    <child link="imu_link"/>
+  </joint>
   <joint name="upper_left_wheel_shaft_joint" type="fixed">
     <origin xyz="0.150 0.108 0.0" rpy="0 0 0" />
@@ -60,8 +84,5 @@
       <origin xyz="0 0.01221 0" rpy="0 0 0"/>
       <mass value="0.055"/>
-      <inertia
-        ixx="0.000021370" ixy="0" ixz="0"
-        iyy="0.000009966" iyz="0"
-        izz="0.000021370"/>
+      <inertia ixx="0.000021370" ixy="0" ixz="0" iyy="0.000009966" iyz="0" izz="0.000021370"/>
     </inertial>
   </link>
@@ -88,8 +109,5 @@
       <origin xyz="0 0.01221 0" rpy="0 0 0"/>
       <mass value="0.055"/>
-      <inertia
-        ixx="0.000021370" ixy="0" ixz="0"
-        iyy="0.000009966" iyz="0"
-        izz="0.000021370"/>
+      <inertia ixx="0.000021370" ixy="0" ixz="0" iyy="0.000009966" iyz="0" izz="0.000021370"/>
     </inertial>
   </link>
@@ -116,8 +134,5 @@
       <origin xyz="0 0.01221 0" rpy="0 0 0"/>
       <mass value="0.055"/>
-      <inertia
-        ixx="0.000021370" ixy="0" ixz="0"
-        iyy="0.000009966" iyz="0"
-        izz="0.000021370"/>
+      <inertia ixx="0.000021370" ixy="0" ixz="0" iyy="0.000009966" iyz="0" izz="0.000021370"/>
     </inertial>
   </link>
@@ -144,8 +159,5 @@
       <origin xyz="0 0.01221 0" rpy="0 0 0"/>
       <mass value="0.055"/>
-      <inertia
-        ixx="0.000021370" ixy="0" ixz="0"
-        iyy="0.000009966" iyz="0"
-        izz="0.000021370"/>
+      <inertia ixx="0.000021370" ixy="0" ixz="0" iyy="0.000009966" iyz="0" izz="0.000021370"/>
     </inertial>
   </link>
@@ -174,8 +186,5 @@
       <mass value="0.3844"/>
       <!-- Inertia based on cylinder -->
-      <inertia
-        ixx="0.000324824" ixy="0" ixz="0"
-        iyy="0.000480000" iyz="0"
-        izz="0.000324824"/>
+      <inertia ixx="0.000324824" ixy="0" ixz="0" iyy="0.000480000" iyz="0" izz="0.000324824"/>
     </inertial>
   </link>
@@ -204,8 +213,5 @@
       <mass value="0.3844"/>
       <!-- Inertia based on cylinder -->
-      <inertia
-        ixx="0.000324824" ixy="0" ixz="0"
-        iyy="0.000480000" iyz="0"
-        izz="0.000324824"/>
+      <inertia ixx="0.000324824" ixy="0" ixz="0" iyy="0.000480000" iyz="0" izz="0.000324824"/>
     </inertial>
   </link>
@@ -234,8 +240,5 @@
       <mass value="0.3844"/>
       <!-- Inertia based on cylinder -->
-      <inertia
-        ixx="0.000324824" ixy="0" ixz="0"
-        iyy="0.000480000" iyz="0"
-        izz="0.000324824"/>
+      <inertia ixx="0.000324824" ixy="0" ixz="0" iyy="0.000480000" iyz="0" izz="0.000324824"/>
     </inertial>
   </link>
@@ -264,8 +267,5 @@
       <mass value="0.3844"/>
       <!-- Inertia based on cylinder -->
-      <inertia
-        ixx="0.000324824" ixy="0" ixz="0"
-        iyy="0.000480000" iyz="0"
-        izz="0.000324824"/>
+      <inertia ixx="0.000324824" ixy="0" ixz="0" iyy="0.000480000" iyz="0" izz="0.000324824"/>
     </inertial>
   </link>
@@ -329,12 +329,8 @@
   <xacro:include filename="$(find nexus_4wd_mecanum_description)/urdf/nexus_4wd_mecanum.gazebo" />
   <!-- Include URM04 ultrasonic range finders -->
-  <xacro:include filename="$(find nexus_4wd_mecanum_description)/urdf/urm04_sensor.xacro"/>
-  <!-- front sensor -->
+  <!-- <xacro:include filename="$(find nexus_4wd_mecanum_description)/urdf/urm04_sensor.xacro"/>
   <xacro:urm04_sensor frame_name="front_sensor" ros_topic="front_sensor" update_rate="10" min_range="0.04" max_range="2.5" horizontal_field_of_view="1.04" vertical_field_of_view="0.04" ray_count="2" />
-  <!-- left sensor -->
   <xacro:urm04_sensor frame_name="left_sensor" ros_topic="left_sensor" update_rate="10" min_range="0.04" max_range="2.5" horizontal_field_of_view="1.04" vertical_field_of_view="0.04" ray_count="2" />
-  <!-- right sensor -->
   <xacro:urm04_sensor frame_name="right_sensor" ros_topic="right_sensor" update_rate="10" min_range="0.04" max_range="2.5" horizontal_field_of_view="1.04" vertical_field_of_view="0.04" ray_count="2" />
-  <!-- rear sensor -->
-  <xacro:urm04_sensor frame_name="rear_sensor" ros_topic="rear_sensor" update_rate="10" min_range="0.04" max_range="2.5" horizontal_field_of_view="1.04" vertical_field_of_view="0.04" ray_count="2" />
+  <xacro:urm04_sensor frame_name="rear_sensor" ros_topic="rear_sensor" update_rate="10" min_range="0.04" max_range="2.5" horizontal_field_of_view="1.04" vertical_field_of_view="0.04" ray_count="2" /> -->
 </robot>
