Commit message: fix the tf bug, now the world frame will be publish by odom, and the tf between robot and world will auto pub and update

File: nexus_4wd_mecanum_description/urdf/livox_mid360.xacro (robot description, xacro)
@@ -23,5 +23,5 @@
                 </geometry>
             </visual>
-            <collision>
+            <!-- <collision>
                 <origin xyz="0 0 0" rpy="0 0 0"/>
                 <geometry>
@@ -30,5 +30,5 @@
                     </box>
                 </geometry>
-            </collision>
+            </collision> -->
         </link>
         <!-- Gazebo 配置 -->

File: nexus_4wd_mecanum_description/urdf/nexus_4wd_mecanum.xacro (robot description, xacro)
@@ -3,4 +3,7 @@
   xmlns:xacro="http://ros.org/wiki/xacro">
   <xacro:property name="namespace" value="$(arg namespace)"/>
+  <xacro:property name="pose_x" value="$(arg pose_x)"/>
+  <xacro:property name="pose_y" value="$(arg pose_y)"/>
+  <xacro:property name="pose_yaw" value="$(arg pose_yaw)"/>
   <xacro:property name="PI" value="3.1415926535897931" />
   <xacro:property name="wheel_radius" value="0.050" />
@@ -35,5 +38,5 @@
         <mesh filename="package://nexus_4wd_mecanum_description/meshes/nexus_base_link.STL" scale="0.001 0.001 0.001"/>
       </geometry>
-      <material name="yellow" />
+      <material name="light_grey" />
     </visual>
     <collision>

Commit message: add px4_sim in launch file

File: nexus_4wd_mecanum_description/urdf/livox_mid360.xacro (robot description, xacro)
@@ -8,5 +8,5 @@
     <xacro:property name="laser_min_range" value="0.1"/>
     <xacro:property name="laser_max_range" value="40"/>
-    <xacro:property name="samples" value="10000"/>
+    <xacro:property name="samples" value="8000"/>
     <xacro:property name="downsample" value="1"/>
     <xacro:macro name="laser_livox" params="NS">

Commit message: 将激光雷达的颜色设置为红色 扩大了柱子世界，增加了一个世界

File: nexus_4wd_mecanum_description/urdf/livox_mid360.xacro (robot description, xacro)
@@ -34,5 +34,5 @@
         <!-- Gazebo 配置 -->
         <gazebo reference="laser_link">
-            <material>Gazebo/Gray</material>
+            <material>Gazebo/Red</material>
             <!--define sensor-->
             <sensor type="ray" name="laser_livox">
